File: pcb/apricot-mem.kicad_sch (KiCad schematic)
At the start: 27 parts, among them J101 Apricot XI Expansion slot, J102 GAL16V8, J103 IO Expansion, U101 74LS573, U102 74LS573, U103 74LS573, U104 74LS245, U105 74LS245, U106 IS65C51216

Commit message: fixing r1.3
Parts:
- added TP108: ~{BHE}, TestPoint:TestPoint_Pad_1.0x1.0mm, symbol Connector:TestPoint_Probe
- added TP109: A0, TestPoint:TestPoint_Pad_1.0x1.0mm, symbol Connector:TestPoint_Probe
- TP103: value I1 -> ~{MEMCS}
Connections:
- net A0: now also TP109.1
- net EXP.SPARE: no longer J102.18 (IO2)
- net MEM.~{CS1}: now also TP103.1
- net MRDY: now also J102.18 (IO2)
- net ~{CLK5}: now also J102.1 (I1/CLK)
- net ~{UB}: now also TP108.1
Other:
- title: Apricot Xi Memory -> Apricot Xi Memory and IO Card

Commit message: r1.3.2 working revision
Parts:
- removed TP102: MRDY, TestPoint:TestPoint_Pad_1.0x1.0mm, symbol Connector:TestPoint_Probe
- C101, C102, C103, C104, C105, C106, C107, C108: value 100n/0.1u PWR -> (none); footprint Capacitor_SMD:C_1206_3216Metric_Pad1.33x1.80mm_HandSolder -> (none)
- CP101: value PPWR -> (none); footprint Capacitor_Tantalum_SMD:CP_EIA-7343-31_Kemet-D -> (none)
- J101: value Apricot XI Expansion slot -> (none); footprint Connector_DIN:DIN41612_B_2x32_Male_Horizontal_THT -> (none)
- J102: value GAL16V8 -> (none); footprint Package_DIP:DIP-20_W7.62mm_Socket -> (none)
- J103: value IO Expansion -> (none); footprint Connector_PinHeader_2.54mm:PinHeader_2x10_P2.54mm_Horizontal -> (none)
- R101: value ~{MWTC} -> (none); footprint Resistor_SMD:R_0603_1608Metric_Pad0.98x0.95mm_HandSolder -> (none)
- R102: value ALE -> (none); footprint Resistor_SMD:R_0603_1608Metric_Pad0.98x0.95mm_HandSolder -> (none)
- TP101: value ALE -> (none); footprint TestPoint:TestPoint_Pad_1.0x1.0mm -> (none)
- TP103: value ~{MEMCS} -> (none); footprint TestPoint:TestPoint_Pad_1.0x1.0mm -> (none)
- TP104: value ~{MRDC} -> (none); footprint TestPoint:TestPoint_Pad_1.0x1.0mm -> (none)
- TP105: value ~{BEN} -> (none); footprint TestPoint:TestPoint_Pad_1.0x1.0mm -> (none)
- TP106: value DT/~{R} -> (none); footprint TestPoint:TestPoint_Pad_1.0x1.0mm -> (none)
- TP107: value ~{MWTC} -> (none); footprint TestPoint:TestPoint_Pad_1.0x1.0mm -> (none)
- TP108: value ~{BHE} -> (none); footprint TestPoint:TestPoint_Pad_1.0x1.0mm -> (none)
- TP109: value A0 -> (none); footprint TestPoint:TestPoint_Pad_1.0x1.0mm -> (none)
- U101, U102, U103: value 74LS573 -> (none); footprint Package_SO:SOIC-20W_7.5x12.8mm_P1.27mm -> (none)
- U104, U105: value 74LS245 -> (none); footprint Package_SO:SOIC-20W_7.5x12.8mm_P1.27mm -> (none)
- U106: value IS65C51216 -> (none); footprint Package_SO:TSOP-II-44_10.16x18.41mm_P0.8mm -> (none)
Connections:
- net EXP.SPARE: now also J102.18 (IO2)
- net MRDY: no longer J102.18 (IO2)
- net ~{CLK5}: no longer J102.1 (I1/CLK)
- no-connect marks 7 -> 8
