File: pcb/apricot-mem.kicad_pcb (KiCad board)
At the start: 2 copper layers, 99.7 x 70 mm, 27 parts, among them J101 Apricot XI Expansion slot, J102 GAL16V8, J103 IO Expansion, U101 74LS573, U102 74LS573, U103 74LS573, U104 74LS245, U105 74LS245, U106 IS65C51216

Commit message: r1.3.2 working revision
Parts:
- removed TP102: MRDY, TestPoint:TestPoint_Pad_1.0x1.0mm
- removed TP103: I1, TestPoint:TestPoint_Pad_1.0x1.0mm
- C101, C102, C103, C104, C105, C106, C107, C108: value 100n/0.1u PWR -> 1uF PWR
Connections:
- J102 pad 1: Net-(J102-Pad1) -> unconnected-(J102-Pad1)
Routing:
- net MRDY: track 2.29 -> 0.00 mm
- net Net-(J102-Pad1): track 2.26 -> 0.00 mm
Changed lines of the file:
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@@
   (title_block
     (title "Apricot Xi Memory")
-    (date "2023-04-06")
-    (rev "1.3")
+    (date "2023-04-21")
+    (rev "1.3.2")
     (company "Atsuko Ito")
   )
@@
   (net 105 "A16")
   (net 106 "EXP.~{CS}")
-  (net 107 "Net-(R101-Pad2)")
+  (net 107 "Net-(J101-Padb21)")
   (net 108 "BUS.~{ENABLED}")
   (net 109 "MEM.~{CS1}")
   (net 110 "EXP.SPARE")
   (net 111 "Net-(J101-Pada15)")
-  (net 112 "Net-(J102-Pad1)")
+  (net 112 "unconnected-(J102-Pad1)")
   (footprint "Capacitor_SMD:C_1206_3216Metric_Pad1.33x1.80mm_HandSolder" (layer "F.Cu")
     (at 105.283 104.648)
@@
       (effects (font (size 1 1) (thickness 0.15)))
     )
-    (fp_text value "100n/0.1u PWR" (at 0 1.85) (layer "F.Fab")
+    (fp_text value "1uF PWR" (at 0 1.85) (layer "F.Fab")
       (effects (font (size 1 1) (thickness 0.15)))
     )
@@
       (effects (font (size 1 1) (thickness 0.15)))
     )
-    (fp_text value "100n/0.1u PWR" (at 0 1.85 90) (layer "F.Fab")
+    (fp_text value "1uF PWR" (at 0 1.85 90) (layer "F.Fab")
       (effects (font (size 1 1) (thickness 0.15)))
     )
@@
       (effects (font (size 1 1) (thickness 0.15)))
     )
-    (fp_text value "100n/0.1u PWR" (at 0 1.85 90) (layer "F.Fab")
+    (fp_text value "1uF PWR" (at 0 1.85 90) (layer "F.Fab")
       (effects (font (size 1 1) (thickness 0.15)))
     )
@@
       (effects (font (size 1 1) (thickness 0.15)))
     )
-    (fp_text value "100n/0.1u PWR" (at 0 1.85) (layer "F.Fab")
+    (fp_text value "1uF PWR" (at 0 1.85) (layer "F.Fab")
       (effects (font (size 1 1) (thickness 0.15)))
     )
@@
       (effects (font (size 1 1) (thickness 0.15)))
     )
-    (fp_text value "100n/0.1u PWR" (at 0 1.85 90) (layer "F.Fab")
+    (fp_text value "1uF PWR" (at 0 1.85 90) (layer "F.Fab")
       (effects (font (size 1 1) (thickness 0.15)))
     )
@@
       (net 66 "~{IOWC}") (pinfunction "Pin_b20") (pintype "passive"))
     (pad "b21" thru_hole circle (at 50.8 2.54 180) (size 1.55 1.55) (drill 1) (layers *.Cu *.Mask)
-      (net 107 "Net-(R101-Pad2)") (pinfunction "Pin_b21") (pintype "passive"))
+      (net 107 "Net-(J101-Padb21)") (pinfunction "Pin_b21") (pintype "passive"))
     (pad "b22" thru_hole circle (at 53.34 2.54 180) (size 1.55 1.55) (drill 1) (layers *.Cu *.Mask)
       (net 62 "~{DMA1}") (pinfunction "Pin_b22") (pintype "passive"))
@@
       (effects (font (size 1 1) (thickness 0.15)))
     )
-    (fp_text value "100n/0.1u PWR" (at 0 1.85 90) (layer "F.Fab")
+    (fp_text value "1uF PWR" (at 0 1.85 90) (layer "F.Fab")
       (effects (font (size 1 1) (thickness 0.15)))
     )
@@
       (effects (font (size 1 1) (thickness 0.15)))
     )
-    (fp_text value "100n/0.1u PWR" (at 0 1.85 90) (layer "F.Fab")
+    (fp_text value "1uF PWR" (at 0 1.85 90) (layer "F.Fab")
       (effects (font (size 1 1) (thickness 0.15)))
     )
@@
       (effects (font (size 1 1) (thickness 0.15)))
     )
-    (fp_text value "100n/0.1u PWR" (at 0 1.85 90) (layer "F.Fab")
+    (fp_text value "1uF PWR" (at 0 1.85 90) (layer "F.Fab")
       (effects (font (size 1 1) (thickness 0.15)))
     )
@@
     (fp_line (start 8.89 24.19) (end 8.89 -1.33) (layer "F.Fab") (width 0.1))
     (pad "1" thru_hole rect (at 0 0 270) (size 1.6 1.6) (drill 0.8) (layers *.Cu *.Mask)
-      (net 112 "Net-(J102-Pad1)") (pinfunction "I1/CLK") (pintype "input"))
+      (net 112 "unconnected-(J102-Pad1)") (pinfunction "I1/CLK") (pintype "input+no_connect"))
     (pad "2" thru_hole oval (at 0 2.54 270) (size 1.6 1.6) (drill 0.8) (layers *.Cu *.Mask)
       (net 69 "DEN") (pinfunction "I2") (pintype "input"))
@@
     )
   )
-  (footprint "TestPoint:TestPoint_Pad_1.0x1.0mm" (layer "B.Cu")
-    (at 110.871 148.463)
-    (descr "SMD rectangular pad as test Point, square 1.0mm side length")
-    (tags "test point SMD pad rectangle square")
-    (property "Sheetfile" "apricot-mem.kicad_sch")
-    (property "Sheetname" "")
-    (property "exclude_from_bom" "")
-    (attr exclude_from_pos_files exclude_from_bom)
-    (fp_text reference "TP102" (at 0 1.448) (layer "B.SilkS") hide
-      (effects (font (size 1 1) (thickness 0.15)) (justify mirror))
-    )
-    (fp_text value "MRDY" (at -2.794 0) (layer "B.SilkS")
-      (effects (font (size 0.78 0.78) (thickness 0.1)) (justify mirror))
-    )
-    (fp_text user "${REFERENCE}" (at 0 1.45) (layer "B.Fab") hide
-      (effects (font (size 1 1) (thickness 0.15)) (justify mirror))
-    )
-    (fp_line (start -0.7 0.7) (end 0.7 0.7) (layer "B.SilkS") (width 0.12))
-    (fp_line (start -0.7 -0.7) (end -0.7 0.7) (layer "B.SilkS") (width 0.12))
-    (fp_line (start 0.7 0.7) (end 0.7 -0.7) (layer "B.SilkS") (width 0.12))
-    (fp_line (start 0.7 -0.7) (end -0.7 -0.7) (layer "B.SilkS") (width 0.12))
-    (fp_line (start 1 -1) (end 1 1) (layer "B.CrtYd") (width 0.05))
-    (fp_line (start -1 1) (end 1 1) (layer "B.CrtYd") (width 0.05))
-    (fp_line (start -1 1) (end -1 -1) (layer "B.CrtYd") (width 0.05))
-    (fp_line (start 1 -1) (end -1 -1) (layer "B.CrtYd") (width 0.05))
-    (pad "1" smd rect (at 0 0) (size 1 1) (layers "B.Cu" "B.Mask")
-      (net 71 "MRDY") (pinfunction "1") (pintype "passive"))
-  )
   (footprint "Resistor_SMD:R_0603_1608Metric_Pad0.98x0.95mm_HandSolder" (layer "B.Cu")
     (at 113.665 129.159)
@@
       (net 64 "~{MWTC}") (pintype "passive"))
     (pad "2" smd roundrect (at 0.9125 0 270) (size 0.975 0.95) (layers "B.Cu" "B.Paste" "B.Mask") (roundrect_rratio 0.25)
-      (net 107 "Net-(R101-Pad2)") (pintype "passive"))
+      (net 107 "Net-(J101-Padb21)") (pintype "passive"))
     (model "${KICAD6_3DMODEL_DIR}/Resistor_SMD.3dshapes/R_0603_1608Metric.wrl"
       (offset (xyz 0 0 0))
@@
       (rotate (xyz 0 0 0))
     )
-  )
-  (footprint "TestPoint:TestPoint_Pad_1.0x1.0mm" (layer "B.Cu")
-    (at 151.638 92.329 180)
-    (descr "SMD rectangular pad as test Point, square 1.0mm side length")
-    (tags "test point SMD pad rectangle square")
-    (property "Sheetfile" "apricot-mem.kicad_sch")
-    (property "Sheetname" "")
-    (property "exclude_from_bom" "")
-    (attr exclude_from_pos_files exclude_from_bom)
-    (fp_text reference "TP103" (at 0 1.448) (layer "B.SilkS") hide
-      (effects (font (size 1 1) (thickness 0.15)) (justify mirror))
-    )
-    (fp_text value "I1" (at 0 -1.55) (layer "B.Fab") hide
-      (effects (font (size 1 1) (thickness 0.15)) (justify mirror))
-    )
-    (fp_text user "${REFERENCE}" (at 0 1.45) (layer "B.Fab") hide
-      (effects (font (size 1 1) (thickness 0.15)) (justify mirror))
-    )
-    (fp_line (start 0.7 -0.7) (end -0.7 -0.7) (layer "B.SilkS") (width 0.12))
-    (fp_line (start -0.7 -0.7) (end -0.7 0.7) (layer "B.SilkS") (width 0.12))
-    (fp_line (start 0.7 0.7) (end 0.7 -0.7) (layer "B.SilkS") (width 0.12))
-    (fp_line (start -0.7 0.7) (end 0.7 0.7) (layer "B.SilkS") (width 0.12))
-    (fp_line (start -1 1) (end 1 1) (layer "B.CrtYd") (width 0.05))
-    (fp_line (start -1 1) (end -1 -1) (layer "B.CrtYd") (width 0.05))
-    (fp_line (start 1 -1) (end 1 1) (layer "B.CrtYd") (width 0.05))
-    (fp_line (start 1 -1) (end -1 -1) (layer "B.CrtYd") (width 0.05))
-    (pad "1" smd rect (at 0 0 180) (size 1 1) (layers "B.Cu" "B.Mask")
-      (net 112 "Net-(J102-Pad1)") (pinfunction "1") (pintype "passive"))
   )
   (gr_line (start 103.1748 134.366) (end 114.3 134.366) (layer "F.SilkS") (width 0.15))
@@
   (segment (start 63.7032 112.9538) (end 63.7032 137.7442) (width 0.25) (layer "B.Cu") (net 70))
   (segment (start 92.3798 139.7508) (end 93.3196 138.811) (width 0.25) (layer "B.Cu") (net 70))
-  (segment (start 110.871 148.463) (end 110.871 146.177) (width 0.25) (layer "B.Cu") (net 71))
   (segment (start 91.948 135.255) (end 96.647 139.954) (width 0.25) (layer "F.Cu") (net 76))
   (segment (start 119.253 141.859) (end 121.031 143.637) (width 0.25) (layer "F.Cu") (net 76))
@@
   (segment (start 114.7064 142.3416) (end 112.9538 140.589) (width 0.25) (layer "B.Cu") (net 111))
   (segment (start 103.9876 134.8232) (end 110.5408 128.27) (width 0.25) (layer "B.Cu") (net 111))
-  (segment (start 151.638 92.7254) (end 151.5668 92.6542) (width 0.25) (layer "B.Cu") (net 112))
   (segment (start 151.5668 94.8536) (end 151.638 94.7824) (width 0.25) (layer "B.Cu") (net 112))
-  (segment (start 151.638 94.7824) (end 151.638 92.7254) (width 0.25) (layer "B.Cu") (net 112))
   (zone (net 1) (net_name "GND") (layers F&B.Cu) (name "EXP GND") (hatch edge 0.508)
     (connect_pads (clearance 0.508))

Commit message: PCB Revision 1.4
* better ground plane
* link to AISLER
Routing:
- net GND: track 246.1 -> 254.0 mm, vias 51 -> 154
- net A19: track 84.1 -> 85.5 mm
- net 5VDC: track 474.2 -> 472.9 mm
- net ~{IOWC}: track 181.7 -> 182.8 mm
- net A18: track 100.8 -> 101.6 mm
- net IORDY: track 76.7 -> 77.4 mm
- net D8: track 21.0 -> 20.4 mm
- net ~{IORC}: track 168.5 -> 169.1 mm
- net D9: track 21.5 -> 21.0 mm
- net D12: track 29.9 -> 30.5 mm
- net D10: track 22.1 -> 21.6 mm
Other:
- board text added: "Rev 1.4"
- board text removed: "Rev 1.3"
